File: Hardware/Platinen-Layout/test-sensor-platiene/test-sensior-platiene.brd (EAGLE design)
At the start: 40 x 40 mm, 38 parts, among them J10 Flash Programming, J5 Flash Programming, U1 AS72651, U10 4MB Flash, U2 4MB Flash, U5 AS72653, U6 AS72652, U9 IR

Commit message: board is a mess
Parts:
- moved U2 84.7 mm to (48.8, 46.4)
- moved D1 77.5 mm to (42.4, 34.9)
- moved C7 71.2 mm to (36.2, 21.9)
- moved J1 69.3 mm to (20.0, 1.65)
- moved D2 69.2 mm to (28.5, 25.2), turned to 180 degrees
- moved C6 67.9 mm to (36.1, 18.8)
- moved C1 67.5 mm to (21.4, 16.8), turned to 180 degrees
- moved C8 64.8 mm to (24.4, 15.0), turned to 90 degrees
- moved U$2 58.2 mm to (31.4, 10.2), turned to 270 degrees
- moved U10 55.5 mm to (7.43, 46.3)
- moved R1 52.9 mm to (4.39, 6.15)
- moved J5 50.7 mm to (31.9, 36.6)
- moved J10 50.1 mm to (18.7, 47.8)
- moved U$1 49.1 mm to (31.2, 2.98), turned to 270 degrees
- moved C5 48.0 mm to (21.2, 33.8), turned to 90 degrees
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Connections:
- new net N$11: J3.2
- new net N$8: J1.2
- net GND: no longer J1.2, J3.2

Commit message: board is getting there
Parts:
- moved R11 73.8 mm to (25.9, 17.8), flipped to the bottom, turned to 180 degrees
- moved R16 62.9 mm to (24.3, 8.54), flipped to the bottom, turned to 180 degrees
- moved R2 61.0 mm to (11.5, 10.5), turned to 180 degrees
- moved R15 60.9 mm to (24.3, 5.99), flipped to the bottom
- moved R14 59.5 mm to (28.1, 8.51), flipped to the bottom
- moved R10 58.1 mm to (10.0, 9.50), flipped to the bottom, turned to 180 degrees
- moved R13 57.7 mm to (28.1, 6.01), flipped to the bottom, turned to 180 degrees
- moved R9 55.9 mm to (10.0, 7.00), flipped to the bottom
- moved R8 54.9 mm to (14.0, 9.50), flipped to the bottom
- moved R7 52.9 mm to (14.0, 7.00), flipped to the bottom, turned to 180 degrees
- moved R6 48.1 mm to (20.0, 24.0), turned to 180 degrees
- moved R12 45.2 mm to (25.6, 19.8), flipped to the bottom
- moved R5 37.2 mm to (11.5, 21.3), flipped to the bottom
- moved R4 34.8 mm to (11.5, 19.0), flipped to the bottom
- moved D1 32.4 mm to (11.6, 25.0)
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Connections:
- net 3.3V1 renamed XORH-1
- net 3.3V2 renamed XORH-2
- net N$2 renamed XORL-1
- net N$5 renamed XORL-2
Routing:
- net 3.3V: track 0.00 -> 30.0 mm
- net SCL_S: track 0.00 -> 18.9 mm
- net I2C_ENB: track 0.00 -> 17.8 mm
- net SDA_S: track 0.00 -> 6.45 mm
- net XORL-2: track 0.00 -> 5.37 mm
- net XORH-2: track 0.00 -> 5.22 mm
- net GND: track 0.00 -> 4.53 mm

Commit message: board is better
Parts:
- moved R13 30.8 mm to (35.7, 35.8), turned to 90 degrees
- moved R15 28.4 mm to (35.7, 32.0), turned to 270 degrees
- moved R14 27.9 mm to (33.7, 35.8), turned to 270 degrees
- moved R16 25.3 mm to (33.7, 32.0), turned to 90 degrees
- moved U2 22.5 mm to (28.2, 7.60)
- moved J5 21.0 mm to (36.5, 9.00)
- moved U$2 20.0 mm to (29.3, 33.1), turned to 270 degrees
- moved R11 17.4 mm to (24.3, 35.1), turned to 0 degrees
- moved R12 13.3 mm to (24.3, 33.1)
- moved R5 9.22 mm to (4.00, 16.0), turned to 90 degrees
- moved U$1 7.62 mm to (5.00, 11.0)
- moved R4 6.30 mm to (6.00, 16.0), turned to 90 degrees
- moved R10 5.23 mm to (6.40, 5.70), turned to 0 degrees
- moved R7 5.23 mm to (10.4, 3.20), turned to 0 degrees
- moved R8 5.23 mm to (10.4, 5.70), turned to 180 degrees
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Connections:
- removed net N$10: J1.3
- removed net N$8: J1.2
- net 3.3V: now also J1.3
- net GND: now also J1.2
Routing:
- net 3.3V: track 30.0 -> 236.9 mm, vias 0 -> 4
- net SCL_S: track 18.9 -> 0.00 mm
- net I2C_ENB: track 17.8 -> 0.00 mm
- net !CS_EE2: track 0.00 -> 17.3 mm
- net SDA-PI: track 0.00 -> 16.3 mm
- net MISO2: track 0.00 -> 11.5 mm
- net N$1: track 0.00 -> 8.02 mm, vias 0 -> 2
- net SCL-PI: track 0.00 -> 6.84 mm
- net MOSI2: track 0.00 -> 6.63 mm
- net SDA_S: track 6.45 -> 0.00 mm
- net XORL-2: track 5.37 -> 0.00 mm
- net XORH-2: track 5.22 -> 0.00 mm
- net XORH-1: track 0.00 -> 4.85 mm
- net GND: track 4.53 -> 0.00 mm
- net XORL-1: track 0.00 -> 4.40 mm
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
Commit message: board is better2
Parts:
- moved C5 0.30 mm to (20.0, 33.3)
Connections:
- removed net N$11: J3.2
- net GND: now also J3.2
Routing:
- net SCK2: track 3.57 -> 33.2 mm, vias 0 -> 1
- net MOSI2: track 6.63 -> 29.1 mm, vias 0 -> 1
- net !RST-ADDR: track 0.00 -> 22.2 mm, vias 0 -> 2
- net SDA_S: track 0.00 -> 18.5 mm, vias 0 -> 3
- net SDA-SENSOR-2: track 0.00 -> 18.3 mm, vias 0 -> 1
- net SCL_S: track 0.00 -> 16.5 mm, vias 0 -> 4
- net N$3: track 1.15 -> 16.3 mm, vias 1 -> 2
- net MISO2: track 11.5 -> 22.2 mm, vias 0 -> 1
- net !CS_EE2: track 17.3 -> 23.4 mm, vias 0 -> 1
- net GND: track 0.00 -> 5.20 mm, vias 0 -> 2

Commit message: almost done
Routing:
- net SCK: track 0.00 -> 37.3 mm, vias 0 -> 3
- net SDA-PI: track 16.4 -> 51.7 mm
- net SCL-SENSOR-2: track 0.00 -> 25.8 mm, vias 0 -> 1
- net SCL-PI: track 6.84 -> 24.3 mm, vias 0 -> 2
- net MOSI: track 0.00 -> 13.2 mm
- net !CS_EE: track 0.00 -> 10.5 mm, vias 0 -> 1
- net XORH-2: track 0.00 -> 10.2 mm
- net MISO: track 0.00 -> 9.27 mm, vias 0 -> 1
- net 3.3V: track 236.6 -> 243.3 mm, vias 4 -> 5
- net SDA-SENSOR-2: track 18.3 -> 24.6 mm
- net XORL-2: track 0.00 -> 5.92 mm

Commit message: almost done2
Routing:
- net SDA_S: track 18.5 -> 83.4 mm, vias 3 -> 4
- net SDA-PI: track 51.7 -> 93.3 mm, vias 0 -> 1
- net I2C_ENB: track 0.00 -> 20.5 mm, vias 0 -> 2
- net MISO: track 9.27 -> 29.0 mm, vias 1 -> 2
- net SCL_S: track 16.5 -> 36.1 mm, vias 4 -> 5
- net MOSI: track 13.2 -> 28.1 mm, vias 0 -> 1
- net !CS_EE: track 10.5 -> 25.3 mm
- net N$4: track 0.00 -> 8.67 mm, vias 0 -> 2
- net !RST-ADDR: track 22.2 -> 23.1 mm
- net 3.3V: track 243.3 -> 243.8 mm

Commit message: todo ground plane
Routing:
- net SCL-PI: track 24.3 -> 93.9 mm
- net 3.3V: track 243.8 -> 265.0 mm, vias 5 -> 6
- net SCL-SENSOR-1: track 2.75 -> 18.5 mm, vias 0 -> 1
- net SDA-SENSOR-1: track 2.04 -> 16.2 mm, vias 0 -> 3
- net GND: track 5.20 -> 0.00 mm, vias 2 -> 0
- net SDA_S: track 83.4 -> 83.8 mm, vias 4 -> 5
- net SDA-PI: track 93.3 -> 93.4 mm, vias 1 -> 2

Commit message: todo ground plane next try
Parts:
- added U$3, U$4, U$5, U$6, U$7: (no value), M3-Hole:3-2MM-HOLE
- moved R15 3.40 mm to (35.7, 28.6)
- moved R16 3.40 mm to (33.7, 28.6)
- moved R13 2.70 mm to (35.7, 33.1)
- moved R14 2.70 mm to (33.7, 33.1)
- moved R9 0.40 mm to (6.80, 3.20)
Routing:
- net SCL-PI: track 93.9 -> 77.1 mm, vias 2 -> 3
- net XORL-1: track 4.40 -> 7.04 mm
- net 3.3V: track 265.0 -> 264.3 mm, vias 6 -> 7
- net SCK: track 37.3 -> 36.6 mm
