File: Hardware/Platinen-Layout/Sensor-platiene/nanopi-black2-shield.sch (EAGLE design)
At the start: 6 parts, among them IC1 LM1117MP-3.3

Commit message: latex template!!!
Parts:
- removed J3: (no value), 61301021821_Eagle_WR-PHD_rev19a:6130XX11021_61300211021
- added C1, C2: 1.0uF, SparkFun-Capacitors:1.0UF-0603-16V-10%
- added J6: (no value), 61300621821_Eagle_WR-PHD_rev19a:6130XX11821_61300211821
Connections:
- net 3,3V: now also C2.1
- net 5V-1: now also C1.1
- net GND: now also C1.2, C2.2
- net RX: now also J6.2; no longer J3.1
- net TX: now also J6.1; no longer J3.2
Changed lines of the file:
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@@
 <part name="J1" library="61300211821_Eagle_WR-PHD_rev19a" deviceset="6130XX21121_61301021121" device="" package3d_urn="urn:adsk.eagle:package:14805405/2"/>
 <part name="J2" library="61300211821_Eagle_WR-PHD_rev19a" deviceset="6130XX21121_61300621121" device="" package3d_urn="urn:adsk.eagle:package:14805407/2"/>
-<part name="J3" library="61301021821_Eagle_WR-PHD_rev19a" deviceset="6130XX11021_61300211021" device="" package3d_urn="urn:adsk.eagle:package:14805448/2"/>
 <part name="GND1" library="supply1" library_urn="urn:adsk.eagle:library:371" deviceset="GND" device=""/>
 <part name="GND2" library="supply1" library_urn="urn:adsk.eagle:library:371" deviceset="GND" device=""/>
@@
 <part name="SUPPLY28" library="SparkFun-PowerSymbols" deviceset="3.3V" device=""/>
 <part name="GND19" library="supply1" library_urn="urn:adsk.eagle:library:371" deviceset="GND" device=""/>
+<part name="J6" library="61300621821_Eagle_WR-PHD_rev19a" deviceset="6130XX11821_61300211821" device="" package3d_urn="urn:adsk.eagle:package:14805539/2"/>
+<part name="C2" library="SparkFun-Capacitors" deviceset="1.0UF" device="-0603-16V-10%" value="1.0uF"/>
+<part name="C1" library="SparkFun-Capacitors" deviceset="1.0UF" device="-0603-16V-10%" value="1.0uF"/>
 </parts>
 <sheets>
@@
 <instances>
 <instance part="IC1" gate="G$1" x="157.48" y="60.96" smashed="yes">
-<attribute name="NAME" x="160.02" y="53.34" size="1.778" layer="95"/>
-<attribute name="VALUE" x="160.02" y="50.8" size="1.778" layer="96"/>
+<attribute name="NAME" x="147.32" y="66.04" size="1.778" layer="95"/>
+<attribute name="VALUE" x="152.4" y="66.04" size="1.778" layer="96"/>
 </instance>
 <instance part="J1" gate="G$1" x="101.6" y="55.88" smashed="yes" rot="R90">
@@
 <attribute name="VALUE" x="82.78" y="-9.49" size="1.016" layer="96" align="bottom-right"/>
 </instance>
-<instance part="J3" gate="G$1" x="81.28" y="25.4" smashed="yes">
-<attribute name="NAME" x="86.38" y="23.745" size="1.016" layer="95"/>
-<attribute name="VALUE" x="86.12" y="22.34" size="1.016" layer="96"/>
-</instance>
 <instance part="GND1" gate="1" x="157.48" y="48.26" smashed="yes">
 <attribute name="VALUE" x="154.94" y="45.72" size="1.778" layer="96"/>
@@
 <instance part="GND19" gate="1" x="170.18" y="5.08" smashed="yes">
 <attribute name="VALUE" x="167.64" y="2.54" size="1.778" layer="96"/>
+</instance>
+<instance part="J6" gate="G$1" x="86.36" y="25.4" smashed="yes">
+<attribute name="NAME" x="81.48" y="24.478" size="1.016" layer="95" align="bottom-right"/>
+<attribute name="VALUE" x="81.53" y="22.82" size="1.016" layer="96" align="bottom-right"/>
+</instance>
+<instance part="C2" gate="G$1" x="165.1" y="53.34" smashed="yes">
+<attribute name="NAME" x="166.624" y="56.261" size="1.778" layer="95" font="vector"/>
+<attribute name="VALUE" x="166.624" y="51.181" size="1.778" layer="96" font="vector"/>
+</instance>
+<instance part="C1" gate="G$1" x="147.32" y="53.34" smashed="yes">
+<attribute name="NAME" x="148.844" y="56.261" size="1.778" layer="95" font="vector"/>
+<attribute name="VALUE" x="148.844" y="51.181" size="1.778" layer="96" font="vector"/>
 </instance>
 </instances>
@@
 <wire x1="157.48" y1="53.34" x2="157.48" y2="50.8" width="0.1524" layer="91"/>
 <pinref part="GND1" gate="1" pin="GND"/>
+<wire x1="147.32" y1="50.8" x2="157.48" y2="50.8" width="0.1524" layer="91"/>
+<junction x="157.48" y="50.8"/>
+<pinref part="C2" gate="G$1" pin="2"/>
+<wire x1="165.1" y1="50.8" x2="157.48" y2="50.8" width="0.1524" layer="91"/>
+<pinref part="C1" gate="G$1" pin="2"/>
 </segment>
 <segment>
@@
 <segment>
 <pinref part="IC1" gate="G$1" pin="IN"/>
-<wire x1="149.86" y1="60.96" x2="144.78" y2="60.96" width="0.1524" layer="91"/>
+<wire x1="149.86" y1="60.96" x2="147.32" y2="60.96" width="0.1524" layer="91"/>
 <label x="144.78" y="60.96" size="1.27" layer="95" rot="R180" xref="yes"/>
+<wire x1="147.32" y1="60.96" x2="144.78" y2="60.96" width="0.1524" layer="91"/>
+<wire x1="147.32" y1="58.42" x2="147.32" y2="60.96" width="0.1524" layer="91"/>
+<junction x="147.32" y="60.96"/>
+<pinref part="C1" gate="G$1" pin="1"/>
 </segment>
 </net>
@@
 <wire x1="165.1" y1="60.96" x2="170.18" y2="60.96" width="0.1524" layer="91"/>
 <label x="170.18" y="60.96" size="1.27" layer="95" xref="yes"/>
+<pinref part="C2" gate="G$1" pin="1"/>
+<wire x1="165.1" y1="58.42" x2="165.1" y2="60.96" width="0.1524" layer="91"/>
+<junction x="165.1" y="60.96"/>
 </segment>
 </net>
 <net name="TX" class="0">
 <segment>
-<pinref part="J3" gate="G$1" pin="2"/>
-<wire x1="81.28" y1="20.32" x2="81.28" y2="17.78" width="0.1524" layer="91"/>
-<label x="81.28" y="17.78" size="1.27" layer="95" rot="R270" xref="yes"/>
+<label x="83.82" y="17.78" size="1.27" layer="95" rot="R270" xref="yes"/>
+<pinref part="J6" gate="G$1" pin="1"/>
+<wire x1="83.82" y1="17.78" x2="83.82" y2="20.32" width="0.1524" layer="91"/>
 </segment>
 <segment>
@@
 <net name="RX" class="0">
 <segment>
-<pinref part="J3" gate="G$1" pin="1"/>
-<wire x1="83.82" y1="20.32" x2="83.82" y2="17.78" width="0.1524" layer="91"/>
-<label x="83.82" y="17.78" size="1.27" layer="95" rot="R270" xref="yes"/>
-</segment>
-<segment>
+<label x="86.36" y="17.78" size="1.27" layer="95" rot="R270" xref="yes"/>
+<pinref part="J6" gate="G$1" pin="2"/>
+<wire x1="86.36" y1="17.78" x2="86.36" y2="20.32" width="0.1524" layer="91"/>
+</segment>
+<segment>
