File: Hardware/Platinen-Layout/Sensor-platiene.sch (EAGLE design)
At the start: 38 parts, among them J10 Flash Programming, J5 Flash Programming, U1 AS72651, U10 4MB Flash, U2 4MB Flash, U5 AS72653, U6 AS72652

Commit message: new hardware + test code
Parts:
- removed U2: 4MB Flash, SparkFun-IC-Memory:AT25SF041
- added U20: AT25SF041, SparkFun-IC-Memory:AT25SF041
- C1, C5: value 1.0uF -> 10uF
- C3, C6: value 1.0uF -> 100nF
- C4, C8: value 10uF -> 100nF
- U10: value 4MB Flash -> AT25SF041
- renumbered R1 to R7, R2 to R8
Connections:
- net !CS_EE: now also U20.!CS; no longer U2.!CS
- net 3.3V: now also U20.!HOLD(D3), U20.!WP(D2), U20.VCC; no longer U2.!HOLD(D3), U2.!WP(D2), U2.VCC
- net GND: now also U20.GND; no longer U2.GND
- net MISO: now also U20.SO(D1); no longer U2.SO(D1)
- net MOSI: now also U20.SI(D0); no longer U2.SI(D0)
- net SCK: now also U20.SCK; no longer U2.SCK
Other:
- note removed: "decoupling capacitor for every sensor"
- moved on the sheet: AS7261, C6, C8, D1-AS7261, R6
