File: Hardware/Platinen-Layout/Sensor-platiene.brd (EAGLE design)
At the start: 40.2 x 40.1 mm, 43 parts, among them J10 Flash Programming, J5 Flash Programming, U1 AS72651, U10 4MB Flash, U2 4MB Flash, U5 AS72653, U6 AS72652

Commit message: add heatsink to board
Routing:
- net SCL-PI: track 77.4 -> 86.5 mm, vias 3 -> 2
- net SDA-PI: track 86.1 -> 92.8 mm
- net GND: vias 20 -> 120
Other:
- board text added: "I2C Spectral Sensor V 1.1"
- board text removed: "I2C Spectral Sensor V 1.0"

Commit message: new hardware + test code
Parts:
- C1, C5: value 1.0uF -> 10uF
- C3, C6: value 1.0uF -> 100nF
- C4, C8: value 10uF -> 100nF
- U10, U20: value 4MB Flash -> AT25SF041
- renumbered R1 to R7, R2 to R8, U2 to U20
Routing:
- net 3.3V: track 275.2 -> 279.0 mm
- net GND: track 7.61 -> 9.01 mm, vias 120 -> 23
Other:
- board text added: "AS7261"
- board text added: "AS7261 periphery"
- board text added: "AS7265X periphery"

Commit message: latex todo list
Routing:
- net SCL-PI: track 86.5 -> 84.8 mm
- net 3.3V: track 279.0 -> 277.5 mm
- net SCL_S: track 37.9 -> 38.5 mm
Changed lines of the file:
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@@
 <drawing>
 <settings>
-<setting alwaysvectorfont="yes"/>
+<setting alwaysvectorfont="no"/>
 <setting verticaltext="up"/>
 </settings>
 <grid distance="0.1" unitdist="mm" unit="mm" style="dots" multiple="1" display="yes" altdistance="0.1" altunitdist="mm" altunit="mm"/>
 <layers>
-<layer number="1" name="Top" color="4" fill="1" visible="yes" active="yes"/>
-<layer number="16" name="Bottom" color="1" fill="1" visible="no" active="yes"/>
+<layer number="1" name="Top" color="4" fill="1" visible="no" active="yes"/>
+<layer number="16" name="Bottom" color="1" fill="1" visible="yes" active="yes"/>
 <layer number="17" name="Pads" color="2" fill="1" visible="yes" active="yes"/>
 <layer number="18" name="Vias" color="2" fill="1" visible="yes" active="yes"/>
 <layer number="19" name="Unrouted" color="6" fill="1" visible="yes" active="yes"/>
 <layer number="20" name="Dimension" color="24" fill="1" visible="yes" active="yes"/>
-<layer number="21" name="tPlace" color="7" fill="1" visible="yes" active="yes"/>
-<layer number="22" name="bPlace" color="7" fill="1" visible="no" active="yes"/>
-<layer number="23" name="tOrigins" color="15" fill="1" visible="yes" active="yes"/>
-<layer number="24" name="bOrigins" color="15" fill="1" visible="no" active="yes"/>
-<layer number="25" name="tNames" color="7" fill="1" visible="yes" active="yes"/>
-<layer number="26" name="bNames" color="7" fill="1" visible="no" active="yes"/>
-<layer number="27" name="tValues" color="7" fill="1" visible="yes" active="yes"/>
+<layer number="21" name="tPlace" color="7" fill="1" visible="no" active="yes"/>
+<layer number="22" name="bPlace" color="7" fill="1" visible="yes" active="yes"/>
+<layer number="23" name="tOrigins" color="15" fill="1" visible="no" active="yes"/>
+<layer number="24" name="bOrigins" color="15" fill="1" visible="yes" active="yes"/>
+<layer number="25" name="tNames" color="7" fill="1" visible="no" active="yes"/>
+<layer number="26" name="bNames" color="7" fill="1" visible="yes" active="yes"/>
+<layer number="27" name="tValues" color="7" fill="1" visible="no" active="yes"/>
 <layer number="28" name="bValues" color="7" fill="1" visible="no" active="yes"/>
 <layer number="29" name="tStop" color="7" fill="3" visible="no" active="yes"/>
@@
 <layer number="37" name="tTest" color="7" fill="1" visible="no" active="yes"/>
 <layer number="38" name="bTest" color="7" fill="1" visible="no" active="yes"/>
-<layer number="39" name="tKeepout" color="4" fill="11" visible="yes" active="yes"/>
-<layer number="40" name="bKeepout" color="1" fill="11" visible="no" active="yes"/>
-<layer number="41" name="tRestrict" color="4" fill="10" visible="yes" active="yes"/>
-<layer number="42" name="bRestrict" color="1" fill="10" visible="no" active="yes"/>
+<layer number="39" name="tKeepout" color="4" fill="11" visible="no" active="yes"/>
+<layer number="40" name="bKeepout" color="1" fill="11" visible="yes" active="yes"/>
+<layer number="41" name="tRestrict" color="4" fill="10" visible="no" active="yes"/>
+<layer number="42" name="bRestrict" color="1" fill="10" visible="yes" active="yes"/>
 <layer number="43" name="vRestrict" color="2" fill="10" visible="no" active="yes"/>
 <layer number="44" name="Drills" color="7" fill="1" visible="no" active="yes"/>
@@
 <layer number="49" name="Reference" color="7" fill="1" visible="no" active="yes"/>
 <layer number="50" name="dxf" color="7" fill="1" visible="no" active="no"/>
-<layer number="51" name="tDocu" color="7" fill="1" visible="yes" active="yes"/>
-<layer number="52" name="bDocu" color="7" fill="1" visible="no" active="yes"/>
+<layer number="51" name="tDocu" color="7" fill="1" visible="no" active="yes"/>
+<layer number="52" name="bDocu" color="7" fill="1" visible="yes" active="yes"/>
 <layer number="53" name="tGND_GNDA" color="7" fill="9" visible="no" active="no"/>
 <layer number="54" name="bGND_GNDA" color="1" fill="9" visible="no" active="no"/>
@@
 <contactref element="J1" pad="1"/>
 <wire x1="27.1945" y1="34.1" x2="27.1945" y2="36.3055" width="0.1524" layer="16"/>
-<wire x1="6.9" y1="12.9" x2="7.3" y2="12.5" width="0.1524" layer="1"/>
 <via x="6.9" y="12.9" extent="1-16" drill="0.35"/>
 <wire x1="6.9" y1="12.9" x2="6.6945" y2="13.1055" width="0.1524" layer="16"/>
@@
 <wire x1="0.7" y1="33.9" x2="0.7" y2="14.2" width="0.1524" layer="16"/>
 <wire x1="0.7" y1="33.9" x2="1.5" y2="34.7" width="0.1524" layer="16"/>
-<wire x1="7.3" y1="12.5" x2="7.3" y2="13.5" width="0.1524" layer="1"/>
-<wire x1="7.3" y1="13.5" x2="6.9" y2="13.9" width="0.1524" layer="1"/>
-<wire x1="6.9" y1="13.9" x2="2" y2="13.9" width="0.1524" layer="1"/>
 <via x="2" y="13.9" extent="1-16" drill="0.35"/>
 <wire x1="2" y1="13.9" x2="1" y2="13.9" width="0.1524" layer="16"/>
@@
 <wire x1="1.5" y1="34.7" x2="4.25" y2="34.7" width="0.1524" layer="16"/>
 <wire x1="4.25" y1="34.7" x2="7.9" y2="38.35" width="0.1524" layer="16"/>
+<wire x1="2" y1="13.9" x2="5.9" y2="13.9" width="0.1524" layer="1"/>
+<wire x1="5.9" y1="13.9" x2="6.9" y2="12.9" width="0.1524" layer="1"/>
 </signal>
 <signal name="SDA-PI">
@@
 <wire x1="1.2" y1="11.1" x2="1.2" y2="17.7" width="0.3048" layer="1"/>
 <wire x1="3.2" y1="9.1" x2="2.8" y2="9.5" width="0.3048" layer="1"/>
+<wire x1="4" y1="8.3" x2="3.2" y2="9.1" width="0.3048" layer="1"/>
 <wire x1="2.8" y1="9.5" x2="1.2" y2="11.1" width="0.3048" layer="1"/>
 <wire x1="19.15" y1="7" x2="15.54" y2="7" width="0.3048" layer="1"/>
@@
 <wire x1="2.05" y1="16.85" x2="1.2" y2="17.7" width="0.3048" layer="16"/>
 <via x="1.2" y="17.7" extent="1-16" drill="0.35"/>
-<wire x1="2.8" y1="9.5" x2="2.8" y2="8.9" width="0.3048" layer="1"/>
-<wire x1="2.8" y1="8.9" x2="3.6" y2="8.1" width="0.3048" layer="1"/>
+<wire x1="4" y1="8.3" x2="4" y2="7.7" width="0.3048" layer="1"/>
 <via x="4" y="7.7" extent="1-16" drill="0.35"/>
-<wire x1="3.6" y1="8.1" x2="4" y2="7.7" width="0.3048" layer="1"/>
 <wire x1="22.2" y1="12.262" x2="22.4" y2="12.262" width="0.3048" layer="1"/>
 <wire x1="22.4206" y1="12.2826" x2="22.4" y2="12.262" width="0.3048" layer="1"/>
@@
 <wire x1="22.1755375" y1="14.0581" x2="21.8" y2="14.4336375" width="0.3048" layer="1"/>
 <wire x1="12.262" y1="16.262" x2="16.162" y2="16.262" width="0.3048" layer="1"/>
-<wire x1="25.0419" y1="32.1244625" x2="24.7244625" y2="32.4419" width="0.3048" layer="1"/>
-<wire x1="24.7244625" y1="32.4419" x2="24.5581" y2="32.4419" width="0.3048" layer="1"/>
-<wire x1="24.5581" y1="32.4419" x2="22" y2="35" width="0.3048" layer="1"/>
-<wire x1="25.0419" y1="28.6961" x2="25.0419" y2="32.1244625" width="0.3048" layer="1"/>
+<wire x1="25.0419" y1="31.9581" x2="22" y2="35" width="0.3048" layer="1"/>
+<wire x1="25.0419" y1="28.6961" x2="25.0419" y2="31.9581" width="0.3048" layer="1"/>
 <wire x1="16.4" y1="25.5" x2="16.4" y2="28.138" width="0.3048" layer="1"/>
 <wire x1="20.5" y1="17.1" x2="21.4" y2="17.1" width="0.3048" layer="1"/>
@@
 <wire x1="38.05" y1="27.75" x2="38.9" y2="28.6" width="0.3048" layer="16"/>
 <wire x1="35.7" y1="27.75" x2="38.05" y2="27.75" width="0.3048" layer="16"/>
-<wire x1="3.6" y1="8.1" x2="3.6" y2="5.6" width="0.3048" layer="1"/>
-<wire x1="3.6" y1="5.6" x2="5" y2="4.2" width="0.3048" layer="1"/>
-<wire x1="5" y1="4.2" x2="7.5" y2="4.2" width="0.3048" layer="1"/>
-<wire x1="7.5" y1="4.2" x2="7.8" y2="4.5" width="0.3048" layer="1"/>
+<wire x1="4" y1="7.7" x2="4" y2="5.2" width="0.3048" layer="1"/>
+<wire x1="4" y1="5.2" x2="4.7" y2="4.5" width="0.3048" layer="1"/>
+<wire x1="4.7" y1="4.5" x2="7.8" y2="4.5" width="0.3048" layer="1"/>
 <via x="7.8" y="4.5" extent="1-16" drill="0.35"/>
 <wire x1="7.8" y1="4.5" x2="8.5" y2="3.8" width="0.3048" layer="16"/>
@@
 <wire x1="24.265" y1="6.965" x2="24.2" y2="6.9" width="0.1524" layer="16"/>
 <via x="24.2" y="6.9" extent="1-16" drill="0.35"/>
-<wire x1="24.2" y1="6.9" x2="23.4" y2="6.1" width="0.1524" layer="1"/>
-<wire x1="23.4" y1="6.1" x2="22.6" y2="6.1" width="0.1524" layer="1"/>
+<wire x1="24.2" y1="6.9" x2="23.4" y2="6.9" width="0.1524" layer="1"/>
+<wire x1="23.4" y1="6.9" x2="22.6" y2="6.1" width="0.1524" layer="1"/>
 </signal>
 <signal name="!CS_EE">
@@
 <contactref element="R7" pad="1"/>
 <contactref element="U5" pad="9"/>
-<wire x1="12.35" y1="12.5" x2="13.875" y2="14.025" width="0.1524" layer="1"/>
-<wire x1="13.875" y1="14.025" x2="14.55" y2="14.7" width="0.1524" layer="1"/>
-<wire x1="14.55" y1="14.7" x2="14.6" y2="14.7" width="0.1524" layer="1"/>
+<wire x1="12.35" y1="12.5" x2="12.45" y2="12.5" width="0.1524" layer="1"/>
+<wire x1="14.65" y1="14.7" x2="12.45" y2="12.5" width="0.1524" layer="1"/>
+<wire x1="14.6" y1="14.7" x2="14.65" y2="14.7" width="0.1524" layer="1"/>
+<wire x1="14.675" y1="14.725" x2="14.65" y2="14.7" width="0.1524" layer="1"/>
 <via x="14.6" y="14.7" extent="1-16" drill="0.35"/>
 <wire x1="14.6" y1="14.7" x2="17.4" y2="14.7" width="0.1524" layer="16"/>
@@
 <wire x1="17.4" y1="14.7" x2="17.912" y2="14.7" width="0.1524" layer="1"/>
 <wire x1="17.912" y1="14.7" x2="18.7" y2="13.912" width="0.1524" layer="1"/>
-<wire x1="13.875" y1="14.025" x2="12.5" y2="15.4" width="0.1524" layer="1"/>
+<wire x1="14.675" y1="14.725" x2="14" y2="15.4" width="0.1524" layer="1"/>
+<wire x1="14" y1="15.4" x2="12.5" y2="15.4" width="0.1524" layer="1"/>
 <via x="12.5" y="15.4" extent="1-16" drill="0.35"/>
 <wire x1="12.5" y1="15.4" x2="11.15" y2="16.75" width="0.1524" layer="16"/>
