File: Hardware/Platinen-Layout/nanopi-black2-shield.sch (EAGLE design)
At the start: 11 parts, among them IC2 LM3940IT-3.3, X1 RASPI_BOARD_B+#_HDC

Commit message: latex todo list
Other:
- note added: "Prototyping Connectors"
Changed lines of the file:
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@@
 <wire x1="71.12" y1="35.56" x2="71.12" y2="-7.62" width="0.1524" layer="97" style="longdash"/>
 <wire x1="71.12" y1="35.56" x2="71.12" y2="83.82" width="0.1524" layer="97" style="longdash"/>
+<wire x1="170.18" y1="86.36" x2="170.18" y2="-7.62" width="0.1524" layer="97" style="longdash"/>
+<text x="182.88" y="78.74" size="1.778" layer="97">Prototyping Connectors</text>
 </plain>
 <instances>
